Commit message: take major steps to porting

File: src/gazebo/launch/robot.urdf (robot description, URDF)
Before this commit: robot robot, 4 links, 0 joints
Links:
- removed link robot/caster
- removed link robot/chassis
- removed link robot/left_wheel
- removed link robot/right_wheel
- added link base_link, mass 2.0; collision box size=0.13 0.12 0.10; visual mesh filename=package://limo_description/meshes/limo_base_decimated.dae

Commit message: world renders, robot still fixing

File: src/gazebo/launch/robot.urdf (robot description, URDF)
Before this commit: robot limo, 1 links, 0 joints
Links:
- removed link base_link
- added link base_footprint
- added link robot/base_link, mass ${base_mass}; collision box size=${base_x_size} ${base_y_size} ${base_z_size}; visual mesh filename=package://gazebo/meshes/limo_base_decimated.dae scale=1 1 1
Joints:
- added joint base_joint: type fixed, parent base_footprint, child robot/base_link, origin xyz=0.0 0.0 0.15 rpy=0 0 0

Commit message: try a bit more

File: src/gazebo/launch/robot.urdf (robot description, URDF)
Before this commit: robot limo_four_diff, 2 links, 1 joints
Links:
- removed link base_footprint
- added link robot/front_left_wheel; visual mesh 
- added link robot/front_right_wheel; visual mesh 
- added link robot/rear_left_wheel; visual mesh 
- added link robot/rear_right_wheel; visual mesh 
- link robot/base_link: mass ${base_mass} -> None; geometry visual mesh 
Joints:
- removed joint base_joint

Commit message: start over

File: src/gazebo/launch/robot.urdf (robot description, URDF)
Before this commit: robot robot, 5 links, 0 joints
Links:
- removed link robot/base_link
- removed link robot/front_left_wheel
- removed link robot/front_right_wheel
- removed link robot/rear_left_wheel
- removed link robot/rear_right_wheel
- added link robot/caster; visual sphere radius=0.2
- added link robot/chassis; visual mesh 
- added link robot/left_wheel; visual cylinder length=0.2 radius=0.4
- added link robot/right_wheel; visual cylinder length=0.2 radius=0.4

Commit message: add updated urdf

File: src/gazebo/launch/robot.urdf (robot description, URDF)
Before this commit: robot robot, 4 links, 0 joints
Links:
- link robot/chassis: geometry visual mesh filename=https://raw.githubusercontent.com/WilliamZhang20/Robot_Navi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
